Commit message: two wheels are good!

File: src/sheep-sim/urdf/sheep_basic.xacro (robot description, xacro)
@@ -1,138 +1,168 @@
-<?xml version="1.0" ?>
-<robot name="m2wr" xmlns:xacro="https://www.ros.org/wiki/xacro" >
-  <material name="black">
-    <color rgba="0.0 0.0 0.0 1.0"/>
-  </material>
-  <material name="blue">
-    <color rgba="0.203125 0.23828125 0.28515625 1.0"/>
-  </material>
-  <material name="green">
-    <color rgba="0.0 0.8 0.0 1.0"/>
-  </material>
-  <material name="grey">
-    <color rgba="0.2 0.2 0.2 1.0"/>
-  </material>
-  <material name="orange">
-    <color rgba="1.0 0.423529411765 0.0392156862745 1.0"/>
-  </material>
-  <material name="brown">
-    <color rgba="0.870588235294 0.811764705882 0.764705882353 1.0"/>
-  </material>
-  <material name="red">
-    <color rgba="0.80078125 0.12890625 0.1328125 1.0"/>
-  </material>
-  <material name="white">
-    <color rgba="1.0 1.0 1.0 1.0"/>
-  </material>
-  <gazebo reference="link_chassis">
-    <material>Gazebo/Orange</material>
-  </gazebo>
-  <gazebo reference="link_left_wheel">
-    <material>Gazebo/Blue</material>
-  </gazebo>
-  <gazebo reference="link_right_wheel">
-    <material>Gazebo/Blue</material>
-  </gazebo>
-  <link name="link_chassis">
-    <!-- pose and inertial -->
-    <pose>0 0 0.1 0 0 0</pose>
-    <inertial>
-      <mass value="5"/>
-      <origin rpy="0 0 0" xyz="0 0 0.1"/>
-      <inertia ixx="0.0395416666667" ixy="0" ixz="0" iyy="0.106208333333" iyz="0" izz="0.106208333333"/>
-    </inertial>
-    <collision name="collision_chassis">
+<?xml version="1.0"?>
+<robot name="diff_drive" xmlns:xacro="http://www.ros.org/wiki/xacro">
+  <xacro:property name="sheep_plate_radius" value="0.2" />
+  <xacro:property name="sheep_plate_thickness" value="0.05" />
+  <xacro:property name="sheep_plate_height_from_ground" value="0.2" />
+  <xacro:property name="wheel_radius" value="0.06" />
+  <xacro:property name="wheel_thickness" value="0.02" />
+  <!-- Base Link -->
+  <link name="chassis">
+    <visual>
+      <origin xyz="0.0 0.0 ${sheep_plate_height_from_ground}" />
       <geometry>
-        <box size="0.5 0.3 0.07"/>
+        <cylinder radius="${sheep_plate_radius}" length="${sheep_plate_thickness}" />
+      </geometry>
+      <material name="blue" />
+    </visual>
+    <collision>
+      <origin xyz="0.0 0.0 ${sheep_plate_height_from_ground}" />
+      <geometry>
+        <cylinder radius="${sheep_plate_radius}" length="${sheep_plate_thickness}" />
       </geometry>
     </collision>
+    <inertial>
+      <mass value="1.14395" />
+      <inertia
+        ixx="0.126164"
+        ixy="0.0"
+        ixz="0.0"
+        iyy="0.416519"
+        iyz="0.0"
+        izz="0.481014" />
+    </inertial>
+  </link>
+  <!-- left wheel Link -->
+  <link name="left_wheel">
+    <!-- <collision>
+      <origin xyz="${wheel_thickness/2} ${-sheep_plate_height_from_ground} 0.0" rpy="0.0 1.5707 0.0" />
+      <geometry>
+        <sphere radius="${wheel_radius}" />
+      </geometry>
+    </collision> -->
     <visual>
-      <origin rpy="0 0 0" xyz="0 0 0"/>
+      <!-- <origin xyz="${1 + wheel_thickness/2} ${-sheep_plate_height_from_ground} 0.0" -->
+      <!-- rpy="0.0 1.5707 0.0" /> -->
+      <!-- <origin xyz="${wheel_thickness/2} ${-sheep_plate_height_from_ground} 0.0" rpy="0.0 1.5707
+      0.0" /> -->
       <geometry>
-        <box size="0.5 0.3 0.07"/>
+        <cylinder radius="${wheel_radius}" length="${wheel_thickness}" />
       </geometry>
-      <material name="blue"/>
+      <material name="black" />
     </visual>
-    <!-- caster front -->
-    <collision name="caster_front_collision">
-      <origin rpy=" 0 0 0" xyz="0.35 0 -0.05"/>
+    <inertial>
+      <mass value="2" />
+      <inertia ixx="0.145833"
+        ixy="0.0"
+        ixz="0.0"
+        iyy="0.145833"
+        iyz="0.0"
+        izz="0.125" />
+    </inertial>
+  </link>
+  <!-- left wheel Link -->
+  <link name="right_wheel">
+    <!-- <collision>
+      <origin xyz="${wheel_thickness/2} ${-sheep_plate_height_from_ground} 0.0" rpy="0.0 1.5707 0.0" />
       <geometry>
-        <sphere radius="0.05"/>
+        <sphere radius="${wheel_radius}" />
       </geometry>
-      <surface>
-        <friction>
-          <ode>
-            <mu>0</mu>
-            <mu2>0</mu2>
-            <slip1>1.0</slip1>
-            <slip2>1.0</slip2>
-          </ode>
-        </friction>
-      </surface>
-    </collision>
-    <visual name="caster_front_visual">
-      <origin rpy=" 0 0 0" xyz="0.2 0 -0.05"/>
+    </collision> -->
+    <visual>
+      <!-- <origin xyz="${wheel_thickness/2} ${-sheep_plate_height_from_ground} 0.0" rpy="0.0 1.5707
+      0.0" /> -->
+      <!-- <origin xyz="0.0 0.0 0.0" rpy="0.0 1.5707 0.0" /> -->
       <geometry>
-        <sphere radius="0.05"/>
+        <cylinder radius="${wheel_radius}" length="${wheel_thickness}" />
       </geometry>
+      <material name="black" />
     </visual>
-    </link>
-  <!-- Create wheel right -->
-  <link name="link_right_wheel">
     <inertial>
-      <mass value="0.2"/>
-      <origin rpy="0 1.5707 1.5707" xyz="0 0 0"/>
-      <inertia ixx="0.00052666666" ixy="0" ixz="0" iyy="0.00052666666" iyz="0" izz="0.001"/>
+      <mass value="2" />
+      <inertia ixx="0.145833"
+        ixy="0.0"
+        ixz="0.0"
+        iyy="0.145833"
+        iyz="0.0"
+        izz="0.125" />
     </inertial>
-    <collision name="link_right_wheel_collision">
-      <origin rpy="0 1.5707 1.5707" xyz="0 0 0" />
+  </link>
+  <link name="caster">
+    <!-- <collision>
       <geometry>
-        <cylinder length="0.04" radius="0.1"/>
+        <sphere radius="0.2" />
       </geometry>
-    </collision>
-    <visual name="link_right_wheel_visual">
-      <origin rpy="0 1.5707 1.5707" xyz="0 0 0"/>
+    </collision> -->
+    <visual>
       <geometry>
-        <cylinder length="0.04" radius="0.1"/>
+        <sphere radius="0.2" />
       </geometry>
+      <material name="white" />
     </visual>
+    <inertial>
+      <origin xyz="-0.957138 -0 0.2" rpy="0 0 0" />
+      <mass value="0.005" />
+      <inertia
+        ixx="0.1"
+        ixy="0.0"
+        ixz="0.0"
+        iyy="0.1"
+        iyz="0.0"
+        izz="0.1" />
+    </inertial>
   </link>
-  <!--   Joint for right wheel  -->
-  <joint name="joint_right_wheel" type="continuous">
-    <origin rpy="0 0 0" xyz="-0.05 0.15 0"/>
-    <child link="link_right_wheel" />
-    <parent link="link_chassis"/>
-    <axis rpy="0 0 0" xyz="0 1 0"/>
-    <limit effort="10000" velocity="1000"/>
-    <joint_properties damping="1.0" friction="1.0" />
+  <!-- joints -->
+  <joint name="left_wheel_joint" type="continuous">
+    <!-- <origin xyz="${sheep_plate_radius} 0.0 0" rpy="-1.5707 0 0" /> -->
+    <parent link="chassis" />
+    <!-- <origin xyz="0.0 0.0 0.0" rpy="0.0 1.5707 0.0" /> -->
+    <origin xyz="0.0 ${sheep_plate_radius + wheel_thickness/2.0} ${sheep_plate_height_from_ground}"
+      rpy="1.5707 0.0 0.0" />
+    <child link="left_wheel" />
+    <axis xyz="0 0 1" />
+    <dynamics damping="0.2" />
   </joint>
-  <!-- Left Wheel link -->
-  <link name="link_left_wheel">
-    <inertial>
-      <mass value="0.2"/>
-      <origin rpy="0 1.5707 1.5707" xyz="0 0 0"/>
-      <inertia ixx="0.00052666666" ixy="0" ixz="0" iyy="0.00052666666" iyz="0" izz="0.001"/>
-    </inertial>
-    <collision name="link_left_wheel_collision">
-      <origin rpy="0 1.5707 1.5707" xyz="0 0 0" />
-      <geometry>
-        <cylinder length="0.04" radius="0.1"/>
-      </geometry>
-    </collision>
-    <visual name="link_left_wheel_visual">
-      <origin rpy="0 1.5707 1.5707" xyz="0 0 0"/>
-      <geometry>
-        <cylinder length="0.04" radius="0.1"/>
-      </geometry>
-    </visual>
-  </link>
-  <!--   Joint for right wheel  -->
-  <joint name="joint_left_wheel" type="continuous">
-    <origin rpy="0 0 0" xyz="-0.05 -0.15 0"/>
-    <child link="link_left_wheel" />
-    <parent link="link_chassis"/>
-    <axis rpy="0 0 0" xyz="0 1 0"/>
-    <limit effort="10000" velocity="1000"/>
-    <joint_properties damping="1.0" friction="1.0" />
+  <joint name="right_wheel_joint" type="continuous">
+    <!-- <origin xyz="${sheep_plate_radius} 0.0 0" rpy="-1.5707 0 0" /> -->
+    <parent link="chassis" />
+    <!-- <origin xyz="0.0 0.0 0.0" rpy="0.0 1.5707 0.0" /> -->
+    <origin
+      xyz="0.0 ${-(sheep_plate_radius + wheel_thickness/2.0)} ${sheep_plate_height_from_ground}"
+      rpy="1.5707 0.0 0.0" />
+    <child link="right_wheel" />
+    <axis xyz="0 0 1" />
+    <dynamics damping="0.2" />
   </joint>
+  <joint name="caster_joint" type="fixed">
+    <origin xyz="-0.957138 -0 0.2" rpy="0 0 0" />
+    <parent link="chassis" />
+    <child link="caster" />
+  </joint>
+  <!-- caster frontal wheel Link -->
+  <ros2_control name="GazeboSystem" type="system">
+    <hardware>
+      <plugin>gazebo_ros2_control/GazeboSystem</plugin>
+    </hardware>
+    <joint name="left_wheel_joint">
+      <command_interface name="velocity">
+        <param name="min">-1</param>
+        <param name="max">1</param>
+      </command_interface>
+      <state_interface name="position" />
+      <state_interface name="velocity" />
+    </joint>
+    <joint name="right_wheel_joint">
+      <command_interface name="velocity">
+        <param name="min">-1</param>
+        <param name="max">1</param>
+      </command_interface>
+      <state_interface name="position" />
+      <state_interface name="velocity" />
+    </joint>
+  </ros2_control>
+  <gazebo>
+    <!-- Joint state publisher -->
+    <plugin filename="libgazebo_ros2_control.so" name="gazebo_ros2_control">
+      <parameters>$(find sheep-sim)/config/diff_drive_controller.yaml</parameters>
+    </plugin>
+  </gazebo>
 </robot>

Commit message: sim is working

File: src/sheep-sim/urdf/sheep_basic.xacro (robot description, xacro)
@@ -3,5 +3,5 @@
   <xacro:property name="sheep_plate_radius" value="0.2" />
   <xacro:property name="sheep_plate_thickness" value="0.05" />
-  <xacro:property name="sheep_plate_height_from_ground" value="0.2" />
+  <xacro:property name="sheep_plate_height_from_ground" value="0.05" />
   <xacro:property name="wheel_radius" value="0.06" />
   <xacro:property name="wheel_thickness" value="0.02" />
@@ -22,117 +22,93 @@
     </collision>
     <inertial>
-      <mass value="1.14395" />
-      <inertia
-        ixx="0.126164"
-        ixy="0.0"
-        ixz="0.0"
-        iyy="0.416519"
-        iyz="0.0"
-        izz="0.481014" />
+      <mass value="3.0" />
+      <inertia ixx="${0.25 * sheep_plate_radius**2 + 1/12 * sheep_plate_thickness**2}"
+        iyy="${0.25 * sheep_plate_radius**2 + 1/12 * sheep_plate_thickness**2}"
+        izz="${0.5 * sheep_plate_radius**2}"
+        ixy="0.0" ixz="0.0" iyz="0.0" />
     </inertial>
   </link>
+  <xacro:macro name="wheel_shape">
+    <geometry>
+      <cylinder radius="${wheel_radius}" length="${wheel_thickness}" />
+    </geometry>
+  </xacro:macro>
   <!-- left wheel Link -->
   <link name="left_wheel">
-    <!-- <collision>
-      <origin xyz="${wheel_thickness/2} ${-sheep_plate_height_from_ground} 0.0" rpy="0.0 1.5707 0.0" />
-      <geometry>
-        <sphere radius="${wheel_radius}" />
-      </geometry>
-    </collision> -->
+    <collision>
+      <xacro:wheel_shape />
+    </collision>
     <visual>
-      <!-- <origin xyz="${1 + wheel_thickness/2} ${-sheep_plate_height_from_ground} 0.0" -->
-      <!-- rpy="0.0 1.5707 0.0" /> -->
-      <!-- <origin xyz="${wheel_thickness/2} ${-sheep_plate_height_from_ground} 0.0" rpy="0.0 1.5707
-      0.0" /> -->
-      <geometry>
-        <cylinder radius="${wheel_radius}" length="${wheel_thickness}" />
-      </geometry>
+      <xacro:wheel_shape />
       <material name="black" />
     </visual>
     <inertial>
-      <mass value="2" />
-      <inertia ixx="0.145833"
-        ixy="0.0"
-        ixz="0.0"
-        iyy="0.145833"
-        iyz="0.0"
-        izz="0.125" />
+      <mass value="1.0" />
+      <inertia ixx="${0.25 * wheel_radius**2 + 1/12 * wheel_thickness**2}"
+        iyy="${0.25 * wheel_radius**2 + 1/12 * wheel_thickness**2}"
+        izz="${0.5 * wheel_radius**2}"
+        ixy="0.0" ixz="0.0" iyz="0.0" />
     </inertial>
   </link>
   <!-- left wheel Link -->
   <link name="right_wheel">
-    <!-- <collision>
-      <origin xyz="${wheel_thickness/2} ${-sheep_plate_height_from_ground} 0.0" rpy="0.0 1.5707 0.0" />
-      <geometry>
-        <sphere radius="${wheel_radius}" />
-      </geometry>
-    </collision> -->
+    <collision>
+      <xacro:wheel_shape />
+    </collision>
     <visual>
-      <!-- <origin xyz="${wheel_thickness/2} ${-sheep_plate_height_from_ground} 0.0" rpy="0.0 1.5707
-      0.0" /> -->
-      <!-- <origin xyz="0.0 0.0 0.0" rpy="0.0 1.5707 0.0" /> -->
-      <geometry>
-        <cylinder radius="${wheel_radius}" length="${wheel_thickness}" />
-      </geometry>
+      <xacro:wheel_shape />
       <material name="black" />
     </visual>
     <inertial>
-      <mass value="2" />
-      <inertia ixx="0.145833"
-        ixy="0.0"
-        ixz="0.0"
-        iyy="0.145833"
-        iyz="0.0"
-        izz="0.125" />
+      <mass value="1.0" />
+      <inertia ixx="${0.25 * wheel_radius**2 + 1/12 * wheel_thickness**2}"
+        iyy="${0.25 * wheel_radius**2 + 1/12 * wheel_thickness**2}"
+        izz="${0.5 * wheel_radius**2}"
+        ixy="0.0" ixz="0.0" iyz="0.0" />
     </inertial>
   </link>
   <link name="caster">
-    <!-- <collision>
+    <collision>
       <geometry>
-        <sphere radius="0.2" />
+        <sphere radius="${wheel_radius/4}" />
       </geometry>
-    </collision> -->
+    </collision>
     <visual>
       <geometry>
-        <sphere radius="0.2" />
+        <sphere radius="${wheel_radius/4}" />
       </geometry>
       <material name="white" />
     </visual>
     <inertial>
-      <origin xyz="-0.957138 -0 0.2" rpy="0 0 0" />
-      <mass value="0.005" />
-      <inertia
-        ixx="0.1"
-        ixy="0.0"
-        ixz="0.0"
-        iyy="0.1"
-        iyz="0.0"
-        izz="0.1" />
+      <mass value="0.01" />
+      <inertia ixx="${2/5 * 0.2 * (wheel_radius/4)**2}"
+        iyy="${2/5 * 0.2 * (wheel_radius/4)**2}"
+        izz="${2/5 * 0.2 * (wheel_radius/4)**2}"
+        ixy="0.0" ixz="0.0" iyz="0.0" />
     </inertial>
   </link>
   <!-- joints -->
   <joint name="left_wheel_joint" type="continuous">
-    <!-- <origin xyz="${sheep_plate_radius} 0.0 0" rpy="-1.5707 0 0" /> -->
     <parent link="chassis" />
-    <!-- <origin xyz="0.0 0.0 0.0" rpy="0.0 1.5707 0.0" /> -->
-    <origin xyz="0.0 ${sheep_plate_radius + wheel_thickness/2.0} ${sheep_plate_height_from_ground}"
-      rpy="1.5707 0.0 0.0" />
     <child link="left_wheel" />
+    <origin
+      xyz="-0.05 ${sheep_plate_radius + wheel_thickness/2.0} ${sheep_plate_height_from_ground}"
+      rpy="-1.5707 0.0 0.0" />
     <axis xyz="0 0 1" />
     <dynamics damping="0.2" />
   </joint>
   <joint name="right_wheel_joint" type="continuous">
-    <!-- <origin xyz="${sheep_plate_radius} 0.0 0" rpy="-1.5707 0 0" /> -->
     <parent link="chassis" />
-    <!-- <origin xyz="0.0 0.0 0.0" rpy="0.0 1.5707 0.0" /> -->
+    <child link="right_wheel" />
     <origin
-      xyz="0.0 ${-(sheep_plate_radius + wheel_thickness/2.0)} ${sheep_plate_height_from_ground}"
-      rpy="1.5707 0.0 0.0" />
-    <child link="right_wheel" />
+      xyz="-0.05 ${-(sheep_plate_radius + wheel_thickness/2.0)} ${sheep_plate_height_from_ground}"
+      rpy="-1.5707 0.0 0.0" />
     <axis xyz="0 0 1" />
     <dynamics damping="0.2" />
   </joint>
   <joint name="caster_joint" type="fixed">
-    <origin xyz="-0.957138 -0 0.2" rpy="0 0 0" />
+    <origin
+      xyz="${sheep_plate_radius*0.75} 0.0 ${sheep_plate_height_from_ground - sheep_plate_thickness/2 - wheel_radius/4}"
+      rpy="0 0 0" />
     <parent link="chassis" />
     <child link="caster" />

Commit message: working sim with field and lidar

File: src/sheep-sim/urdf/sheep_basic.xacro (robot description, xacro)
@@ -81,9 +81,29 @@
     </visual>
     <inertial>
-      <mass value="0.01" />
+      <mass value="0.1" />
       <inertia ixx="${2/5 * 0.2 * (wheel_radius/4)**2}"
         iyy="${2/5 * 0.2 * (wheel_radius/4)**2}"
         izz="${2/5 * 0.2 * (wheel_radius/4)**2}"
         ixy="0.0" ixz="0.0" iyz="0.0" />
+    </inertial>
+  </link>
+  <link name="lidar_link">
+    <visual>
+      <origin xyz="0 0 0" rpy="0 0 0" />
+      <geometry>
+        <cylinder length="0.05" radius="0.05" />
+      </geometry>
+      <material name="silver" />
+    </visual>
+    <collision>
+      <origin xyz="0 0 0" rpy="0 0 0" />
+      <geometry>
+        <cylinder length="0.05" radius="0.05" />
+      </geometry>
+    </collision>
+    <inertial>
+      <origin xyz="0 0 0" rpy="0 0 0" />
+      <mass value="0.005" />
+      <inertia ixx="0.0001" iyy="0.0001" izz="0.0001" ixy="0" ixz="0" iyz="0" />
     </inertial>
   </link>
@@ -113,4 +133,9 @@
     <parent link="chassis" />
     <child link="caster" />
+  </joint>
+  <joint name="lidar_joint" type="fixed">
+    <parent link="chassis" />
+    <child link="lidar_link" />
+    <origin xyz="0 0 ${sheep_plate_height_from_ground + sheep_plate_thickness + 0.02}" rpy="0 0 0" />
   </joint>
   <!-- caster frontal wheel Link -->
@@ -140,5 +165,43 @@
     <plugin filename="libgazebo_ros2_control.so" name="gazebo_ros2_control">
       <parameters>$(find sheep-sim)/config/diff_drive_controller.yaml</parameters>
+      <!-- <ros>
+      <remapping>~/diff_drive_base_controller/cmd_vel_unstamped:=cmd_vel</remapping>
+    </ros> -->
     </plugin>
   </gazebo>
+  <gazebo reference="lidar_link">
+    <sensor type="ray" name="lidar_sensor">
+      <pose>0 0 0 0 0 0</pose>
+      <visualize>true</visualize>
+      <update_rate>10</update_rate>
+      <ray>
+        <scan>
+          <horizontal>
+            <samples>360</samples>
+            <resolution>1</resolution>
+            <min_angle>0.0000000</min_angle>
+            <max_angle>6.28</max_angle>
+          </horizontal>
+        </scan>
+        <range>
+          <min>0.1</min>
+          <max>30</max>
+          <resolution>0.01</resolution>
+        </range>
+        <noise>
+          <type>gaussian</type>
+          <mean>0.0</mean>
+          <stddev>0.01</stddev>
+        </noise>
+      </ray>
+      <plugin name="scan" filename="libgazebo_ros_ray_sensor.so">
+        <!-- <ros>
+          <remapping>~/out:=scan</remapping>
+        </ros> -->
+        <!-- <topicName>/scan</topicName> -->
+        <output_type>sensor_msgs/LaserScan</output_type>
+        <frameName>lidar_link</frameName>
+      </plugin>
+    </sensor>
+  </gazebo>
 </robot>

Commit message: movement is great

File: src/sheep-sim/urdf/sheep_basic.xacro (robot description, xacro)
@@ -8,4 +8,15 @@
   <!-- Base Link -->
   <link name="chassis">
+  </link>
+  <macro name="cylinder_inertia" params="m r h">
+    <inertial>
+      <mass value="${m}" />
+      <inertia ixx="${m*(3*r*r+h*h)/12}" ixy="0" ixz="0"
+        iyy="${m*(3*r*r+h*h)/12}" iyz="0"
+        izz="${m*r*r/2}"
+      />
+    </inertial>
+  </macro>
+  <link name="base_footprint">
     <visual>
       <origin xyz="0.0 0.0 ${sheep_plate_height_from_ground}" />
@@ -21,5 +32,5 @@
       </geometry>
     </collision>
-    <inertial>
+    <!-- <inertial>
       <mass value="3.0" />
       <inertia ixx="${0.25 * sheep_plate_radius**2 + 1/12 * sheep_plate_thickness**2}"
@@ -27,5 +38,6 @@
         izz="${0.5 * sheep_plate_radius**2}"
         ixy="0.0" ixz="0.0" iyz="0.0" />
-    </inertial>
+    </inertial> -->
+    <xacro:cylinder_inertia m="10" r="${sheep_plate_radius}" h="${sheep_plate_thickness}" />
   </link>
   <xacro:macro name="wheel_shape">
@@ -43,5 +55,6 @@
       <material name="black" />
     </visual>
-    <inertial>
+    <xacro:cylinder_inertia m="10" r="${wheel_radius}" h="${wheel_thickness}" />
+    <!-- <inertial>
       <mass value="1.0" />
       <inertia ixx="${0.25 * wheel_radius**2 + 1/12 * wheel_thickness**2}"
@@ -49,5 +62,5 @@
         izz="${0.5 * wheel_radius**2}"
         ixy="0.0" ixz="0.0" iyz="0.0" />
-    </inertial>
+    </inertial> -->
   </link>
   <!-- left wheel Link -->
@@ -60,5 +73,6 @@
       <material name="black" />
     </visual>
-    <inertial>
+    <xacro:cylinder_inertia m="10" r="${wheel_radius}" h="${wheel_thickness}" />
+    <!-- <inertial>
       <mass value="1.0" />
       <inertia ixx="${0.25 * wheel_radius**2 + 1/12 * wheel_thickness**2}"
@@ -66,5 +80,5 @@
         izz="${0.5 * wheel_radius**2}"
         ixy="0.0" ixz="0.0" iyz="0.0" />
-    </inertial>
+    </inertial> -->
   </link>
   <link name="caster">
@@ -73,4 +87,14 @@
         <sphere radius="${wheel_radius/4}" />
       </geometry>
+      <surface>
+        <friction>
+          <ode>
+            <mu>0.01</mu>
+            <mu2>0.01</mu2>
+            <slip1>1.00</slip1>
+            <slip2>1.00</slip2>
+          </ode>
+        </friction>
+      </surface>
     </collision>
     <visual>
@@ -82,7 +106,11 @@
     <inertial>
       <mass value="0.1" />
-      <inertia ixx="${2/5 * 0.2 * (wheel_radius/4)**2}"
-        iyy="${2/5 * 0.2 * (wheel_radius/4)**2}"
-        izz="${2/5 * 0.2 * (wheel_radius/4)**2}"
+      <!-- <inertia ixx="${2/5 * 0.2 * (wheel_radius/4)**2}"
+      iyy="${2/5 * 0.2 * (wheel_radius/4)**2}"
+      izz="${2/5 * 0.2 * (wheel_radius/4)**2}"
+      ixy="0.0" ixz="0.0" iyz="0.0" /> -->
+      <inertia ixx="0.001"
+        iyy="0.001"
+        izz="0.001"
         ixy="0.0" ixz="0.0" iyz="0.0" />
     </inertial>
@@ -113,5 +141,5 @@
     <child link="left_wheel" />
     <origin
-      xyz="-0.05 ${sheep_plate_radius + wheel_thickness/2.0} ${sheep_plate_height_from_ground}"
+      xyz="-0.09 ${sheep_plate_radius + wheel_thickness/2.0} ${sheep_plate_height_from_ground}"
       rpy="-1.5707 0.0 0.0" />
     <axis xyz="0 0 1" />
@@ -122,5 +150,5 @@
     <child link="right_wheel" />
     <origin
-      xyz="-0.05 ${-(sheep_plate_radius + wheel_thickness/2.0)} ${sheep_plate_height_from_ground}"
+      xyz="-0.09 ${-(sheep_plate_radius + wheel_thickness/2.0)} ${sheep_plate_height_from_ground}"
       rpy="-1.5707 0.0 0.0" />
     <axis xyz="0 0 1" />
@@ -134,8 +162,12 @@
     <child link="caster" />
   </joint>
+  <joint name="base_footprint_joint" type="fixed">
+    <parent link="chassis" />
+    <child link="base_footprint" />
+  </joint>
   <joint name="lidar_joint" type="fixed">
     <parent link="chassis" />
     <child link="lidar_link" />
-    <origin xyz="0 0 ${sheep_plate_height_from_ground + sheep_plate_thickness + 0.02}" rpy="0 0 0" />
+    <origin xyz="0 0 ${sheep_plate_height_from_ground + sheep_plate_thickness + 0.02 }" rpy="0 0 0" />
   </joint>
   <!-- caster frontal wheel Link -->
