Commit message: many changes, idk

File: src/sheep-sim/urdf/sheep_basic.xacro (robot description, xacro)
@@ -7,5 +7,14 @@
   <xacro:property name="wheel_thickness" value="0.02" />
   <!-- Base Link -->
-  <link name="chassis">
+  <xacro:macro name="cylinder_inertia" params="m r h">
+    <inertial>
+      <mass value="${m}" />
+      <inertia ixx="${m*(3*r*r+h*h)/12}" ixy="0" ixz="0"
+        iyy="${m*(3*r*r+h*h)/12}" iyz="0"
+        izz="${m*r*r/2}"
+      />
+    </inertial>
+  </xacro:macro>
+  <link name="base_footprint">
     <visual>
       <origin xyz="0.0 0.0 ${sheep_plate_height_from_ground}" />
@@ -142,3 +151,38 @@
     </plugin>
   </gazebo>
+  <gazebo reference="lidar_link">
+    <sensor type="ray" name="lidar_sensor">
+      <pose>0 0 0 0 0 0</pose>
+      <visualize>true</visualize>
+      <update_rate>10</update_rate>
+      <ray>
+        <scan>
+          <horizontal>
+            <samples>360</samples>
+            <resolution>1</resolution>
+            <min_angle>0.0000000</min_angle>
+            <max_angle>6.28</max_angle>
+          </horizontal>
+        </scan>
+        <range>
+          <min>0.1</min>
+          <max>30</max>
+          <resolution>0.01</resolution>
+        </range>
+        <noise>
+          <type>gaussian</type>
+          <mean>0.0</mean>
+          <stddev>0.01</stddev>
+        </noise>
+      </ray>
+      <plugin name="scan" filename="libgazebo_ros_ray_sensor.so">
+        <ros>
+          <remapping>~/out:=laserscan</remapping>
+        </ros>
+        <!-- <topicName>/scan</topicName> -->
+        <output_type>sensor_msgs/LaserScan</output_type>
+        <frameName>lidar_link</frameName>
+      </plugin>
+    </sensor>
+  </gazebo>
 </robot>
